Commit message: fix(robots): the reference UGV's NavSat horizontal noise in degrees, not metres
The gnss macro passed the manifest's 1 m horizontal stddev straight into
the NavSat sensor, which applies it to latitude and longitude in degrees,
so the fix wandered by about a degree. The macro converts it (one degree
of latitude is 111.32 km); test_ugv_ref checks the conversion. The fault
injection integration test ignores the CLI's lost-message lines when it
reads a field.

Closes #63
Task: P2-T03

File: robots/fieldproof_robots/models/ugv_ref/urdf/sensors.xacro (robot description, xacro)
@@ -116,5 +116,9 @@
     </gazebo>
   </xacro:macro>
-  <!-- Single-band GNSS: about one metre horizontal and two metres vertical position noise. -->
+  <!-- Single-band GNSS: about one metre horizontal and two metres vertical position noise.
+       The NavSat sensor applies the horizontal noise to the latitude and longitude it outputs,
+       in degrees, so the stddev is converted from metres (one degree of latitude is 111.32 km;
+       the longitude noise comes out a little under a metre east at the depot's latitude). -->
+  <xacro:property name="metres_per_degree" value="111319.49"/>
   <xacro:macro name="gnss" params="link topic rate horizontal_stddev:=1.0 vertical_stddev:=2.0 velocity_stddev:=0.1">
     <gazebo reference="${link}">
@@ -130,5 +134,5 @@
               <noise type="gaussian">
                 <mean>0.0</mean>
-                <stddev>${horizontal_stddev}</stddev>
+                <stddev>${horizontal_stddev / metres_per_degree}</stddev>
               </noise>
             </horizontal>
